File: KiCAD_Custom_DRC_Rules_for_PCBWay.kicad_pcb (KiCad board)
At the start: 2 copper layers, 90 x 80 mm, 38 parts, among them J1 Screw_Terminal_01x02, J2 x2 OpAmp ZIF, J3 x1 OpAmp ZIF, J4 x4 OpAmp ZIF, U1 TL072

Commit message: moving some traces around
Routing:
- net Vneg: track 196.9 -> 213.4 mm
Changed lines of the file:
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@@
 		(tags "SOIC SO")
 		(property "Reference" "U1"
-			(at 0 -3.4 360)
+			(at 0 -3.4 0)
 			(layer "F.SilkS")
 			(effects
@@
 		)
 		(property "Value" "TL072"
-			(at 0 3.4 360)
+			(at 0 3.4 0)
 			(layer "F.Fab")
 			(effects
@@
 		)
 		(fp_text user "${REFERENCE}"
-			(at 0 0 360)
+			(at 0 0 0)
 			(layer "F.Fab")
 			(effects
@@
 		(tags "THT DIP DIL CERDIP ceramic 2.54mm 7.62mm 300mil SideBrazed LongPads Socket")
 		(property "Reference" "J3"
-			(at 3.81 -2.965 360)
+			(at 3.81 -2.965 0)
 			(layer "F.SilkS")
 			(effects
@@
 		)
 		(property "Value" "x1 OpAmp ZIF"
-			(at 3.81 18.205 360)
+			(at 3.81 18.205 0)
 			(layer "F.Fab")
 			(effects
@@
 		(tags "resistor")
 		(property "Reference" "R7"
-			(at 0 -1.65 360)
+			(at 0 -1.65 0)
 			(layer "F.SilkS")
 			(effects
@@
 		)
 		(property "Value" "47k"
-			(at 0 1.65 360)
+			(at 0 1.65 0)
 			(layer "F.Fab")
 			(effects
@@
 		)
 		(fp_text user "${REFERENCE}"
-			(at 0 0 360)
+			(at 0 0 0)
 			(layer "F.Fab")
 			(effects
@@
 		(tags "capacitor")
 		(property "Reference" "C3"
-			(at 0 -1.68 360)
+			(at 0 -1.68 0)
 			(layer "F.SilkS")
 			(effects
@@
 		)
 		(property "Value" "0.1uF"
-			(at 0 1.68 360)
+			(at 0 1.68 0)
 			(layer "F.Fab")
 			(effects
@@
 		)
 		(fp_text user "${REFERENCE}"
-			(at 0 0 360)
+			(at 0 0 0)
 			(layer "F.Fab")
 			(effects
@@
 		)
 		(fp_text user "${REFERENCE}"
-			(at 3.81 7.62 360)
+			(at 3.81 7.62 0)
 			(layer "F.Fab")
 			(effects
@@
 		(tags "resistor")
 		(property "Reference" "R10"
-			(at 0 -1.65 360)
+			(at 0 -1.65 0)
 			(layer "F.SilkS")
 			(effects
@@
 		)
 		(property "Value" "1k"
-			(at 0 1.65 360)
+			(at 0 1.65 0)
 			(layer "F.Fab")
 			(effects
@@
 		)
 		(fp_text user "${REFERENCE}"
-			(at 0 0 360)
+			(at 0 0 0)
 			(layer "F.Fab")
 			(effects
@@
 	)
 	(segment
-		(start 109.981051 70.981051)
-		(end 114.401051 70.981051)
+		(start 71.29 71.41)
+		(end 66.582233 71.41)
 		(width 0.5)
 		(layer "B.Cu")
@@
 	)
 	(segment
-		(start 106.58 67.58)
-		(end 75.12 67.58)
+		(start 75.12 67.58)
+		(end 71.29 71.41)
 		(width 0.5)
 		(layer "B.Cu")
@@
 	)
 	(segment
-		(start 81.315 117.92)
-		(end 77.815 117.92)
+		(start 63 74.992233)
+		(end 63 103.105)
 		(width 0.5)
 		(layer "B.Cu")
@@
 	)
 	(segment
-		(start 114.401051 70.981051)
-		(end 119.42 76)
+		(start 81.315 117.92)
+		(end 77.815 117.92)
 		(width 0.5)
 		(layer "B.Cu")
@@
 	)
 	(segment
-		(start 82 118.605)
-		(end 81.315 117.92)
+		(start 63 103.105)
+		(end 77.815 117.92)
 		(width 0.5)
 		(layer "B.Cu")
@@
 	)
 	(segment
-		(start 112.5 122)
-		(end 93 122)
+		(start 82 118.605)
+		(end 81.315 117.92)
 		(width 0.5)
 		(layer "B.Cu")
@@
 	)
 	(segment
-		(start 106.58 67.58)
-		(end 109.981051 70.981051)
+		(start 112.5 122)
+		(end 93 122)
 		(width 0.5)
 		(layer "B.Cu")
@@
 	)
 	(segment
+		(start 66.582233 71.41)
+		(end 63 74.992233)
+		(width 0.5)
+		(layer "B.Cu")
+		(net 3)
+	)
+	(segment
 		(start 119.42 78.42)
 		(end 126 85)
@@
 		(start 118 110.42)
 		(end 118 105.34)
-		(width 0.5)
+		(width 0.75)
 		(layer "F.Cu")
 		(net 38)
@@
 		(start 121.5 110.42)
 		(end 118 110.42)
-		(width 0.5)
+		(width 0.75)
 		(layer "F.Cu")
 		(net 38)
@@
 		(start 118 110.42)
 		(end 113.88 110.42)
-		(width 0.5)
+		(width 0.75)
 		(layer "F.Cu")
 		(net 38)
@@
 		(start 113.88 105.34)
 		(end 118 105.34)
-		(width 0.5)
+		(width 0.75)
 		(layer "F.Cu")
 		(net 38)
@@
 		(start 118 105.34)
 		(end 121.5 105.34)
-		(width 0.5)
+		(width 0.75)
 		(layer "F.Cu")
 		(net 38)
@@
 	)
 	(segment
-		(start 113.5 80)
-		(end 116.88 76.62)
+		(start 90.5 93)
+		(end 100.5 93)
 		(width 0.5)
 		(layer "B.Cu")
@@
 	)
 	(segment
-		(start 90.5 93)
-		(end 103.5 80)
+		(start 100.5 93)
+		(end 116.88 76.62)
 		(width 0.5)
 		(layer "B.Cu")
@@
 		(width 0.5)
 		(layer "B.Cu")
-		(net 38)
-	)
-	(segment
-		(start 103.5 80)
-		(end 113.5 80)
-		(width 0.5)
-		(layer "B.Cu")
