File: KiCAD_Custom_DRC_Rules_for_PCBWay.kicad_pcb (KiCad board)
At the start: 2 copper layers, 90 x 80 mm, 38 parts, among them J1 Screw_Terminal_01x02, J2 x2 OpAmp ZIF, J3 x1 OpAmp ZIF, J4 x4 OpAmp ZIF, U1 TL072

Commit message: cleanup, datasheet updates, add BOM
Parts:
- U1: value TL072 -> TL072H
Routing:
- net Vneg: track 213.4 -> 212.7 mm
Changed lines of the file:
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@@
 			)
 		)
-		(property "Value" "TL072"
+		(property "Value" "TL072H"
 			(at 0 3.4 0)
 			(layer "F.Fab")
@@
 			)
 		)
-		(property "Datasheet" "http://www.ti.com/lit/ds/symlink/tl071.pdf"
+		(property "Datasheet" "https://www.ti.com/lit/ds/symlink/tl072h.pdf"
 			(at 0 0 0)
 			(unlocked yes)
@@
 	)
 	(segment
-		(start 121.88 107.5)
-		(end 121.5 107.88)
-		(width 0.5)
-		(layer "F.Cu")
-		(net 3)
-	)
-	(segment
 		(start 119.5 82.55)
 		(end 119.5 76.08)
@@
 	)
 	(segment
-		(start 119.5 76.08)
-		(end 119.42 76)
-		(width 0.5)
-		(layer "F.Cu")
-		(net 3)
-	)
-	(segment
 		(start 57.315 118.92)
 		(end 72.765 118.92)
@@
 	)
 	(segment
-		(start 111.5 76.3)
-		(end 111.8 76)
-		(width 0.5)
-		(layer "F.Cu")
-		(net 13)
-	)
-	(segment
 		(start 111.5 82.5875)
 		(end 111.5 76.3)
@@
 	)
 	(segment
-		(start 117 68.26)
-		(end 116.88 68.38)
-		(width 0.5)
-		(layer "F.Cu")
-		(net 14)
-	)
-	(segment
 		(start 117 62.4125)
 		(end 117 68.26)
@@
 		(layer "F.Cu")
 		(net 31)
-	)
-	(segment
-		(start 121.74 100.5)
-		(end 121.5 100.26)
-		(width 0.5)
-		(layer "F.Cu")
-		(net 31)
